Commit message: Next steps using a Xacro template

File: ros_ws/src/karaburan.xacro (robot description, xacro)
@@ -1,4 +1,4 @@
 <?xml version="1.0" ?>
-<robot name="karaburan">
+<robot name="karaburan" xmlns:xacro="http://www.ros.org/wiki/xacro">
   <material name="black">
      <color rgba="0.9 0.9 0.9 0.8" />
@@ -23,26 +23,21 @@
     </visual>
   </link>
-  <link name="left_prop">
-    <visual>
-      <geometry>
-        <cylinder radius="0.04" length="0.025" />
-      </geometry>
-      <origin xyz="0 0 0" rpy="0 1.57 0" />
-      <material name="black" />
-    </visual>
-  </link>
-  <link name="right_prop">
-    <visual>
-      <geometry>
-        <cylinder radius="0.04" length="0.025" />
-      </geometry>
-      <origin xyz="0 0 0" rpy="0 1.57 0" />
-      <material name="black" />
-    </visual>
-  </link>
+  <xacro:macro name="prop_link" params="prefix">
+    <link name="${prefix}_prop">
+      <visual>
+        <geometry>
+          <cylinder radius="0.04" length="0.025" />
+        </geometry>
+        <origin xyz="0 0 0" rpy="0 1.57 0" />
+        <material name="black" />
+      </visual>
+    </link>
+  </xacro:macro>
+  <xacro:prop_link prefix="left" />
+  <xacro:prop_link prefix="right" />
   <joint name="base_joint" type="fixed">
     <parent link="base_footprint" />
     <child link="base_link" />
-    <origin xyz="0 -0.1 0" rpy="0 0 0" />
+    <origin xyz="0 0 -0.1" rpy="0 0 0" />
   </joint>
   <joint name="base_lidar_joint" type="fixed">

Commit message: Added basic collision info

File: ros_ws/src/karaburan.xacro (robot description, xacro)
@@ -13,4 +13,10 @@
       <material name="black" />
     </visual>
+    <collision>
+      <geometry>
+        <box size="0.6 0.4 0.2" />
+      </geometry>
+      <origin xyz="0 0 0.1" rpy="0 0 0" />
+    </collision>
   </link>
   <link name="lidar">
@@ -22,4 +28,11 @@
       <material name="black" />
     </visual>
+    <collision>
+      <geometry>
+        <box size="0.1 0.1 0.05" />
+      </geometry>
+      <origin xyz="0 0 0" rpy="0 0 0" />
+      <material name="black" />
+    </collision>
   </link>
   <xacro:macro name="prop_link" params="prefix">

Commit message: Adding imu

File: ros_ws/src/karaburan.xacro (robot description, xacro)
@@ -20,4 +20,15 @@
     </collision>
   </link>
+  <link name="imu">
+    <visual>
+      <geometry>
+        <box size="0.03 0.03 0.001"/>
+      </geometry>
+      <origin xyz="0 0 0" rpy="0 0 0" />
+      <material name="black" />
+    </visual>
+    <collision>
+    </collision>
+  </link>
   <link name="lidar">
     <visual>
@@ -36,4 +47,14 @@
     </collision>
   </link>
+  <joint name="base_joint" type="fixed">
+    <parent link="base_footprint" />
+    <child link="base_link" />
+    <origin xyz="0 0 -0.1" rpy="0 0 0" />
+  </joint>
+  <joint name="base_imu_joint" type="fixed">
+    <parent link="base_link" />
+    <child link="imu" />
+    <origin xyz="0.55 0 0.201" rpy="0 0 0" />
+  </joint>
   <xacro:macro name="prop_link" params="prefix">
     <link name="${prefix}_prop">
@@ -49,9 +70,4 @@
   <xacro:prop_link prefix="left" />
   <xacro:prop_link prefix="right" />
-  <joint name="base_joint" type="fixed">
-    <parent link="base_footprint" />
-    <child link="base_link" />
-    <origin xyz="0 0 -0.1" rpy="0 0 0" />
-  </joint>
   <joint name="base_lidar_joint" type="fixed">
     <parent link="base_link" />

Commit message: Adding GPS and IMU to URDF file

File: ros_ws/src/karaburan.xacro (robot description, xacro)
@@ -31,4 +31,15 @@
     </collision>
   </link>
+  <link name="gps">
+    <visual>
+      <geometry>
+        <box size="0.03 0.03 0.01"/>
+      </geometry>
+      <origin xyz="0 0 0" rpy="0 0 0" />
+      <material name="black" />
+    </visual>
+    <collision>
+    </collision>
+  </link>
   <link name="lidar">
     <visual>
@@ -55,5 +66,10 @@
     <parent link="base_link" />
     <child link="imu" />
-    <origin xyz="0.55 0 0.201" rpy="0 0 0" />
+    <origin xyz="0.25 0 0.201" rpy="0 0 0" />
+  </joint>
+  <joint name="base_gps_joint" type="fixed">
+    <parent link="base_link" />
+    <child link="gps" />
+    <origin xyz="-0.25 0 0.201" rpy="0 0 0" />
   </joint>
   <xacro:macro name="prop_link" params="prefix">
