Commit message: Fixing errors during startup by renaming to magic name imu_link

File: ros_ws/src/navigation/config/karaburan.xacro (robot description, xacro)
@@ -20,5 +20,5 @@
     </collision>
   </link>
-  <link name="imu">
+  <link name="imu_link">
     <visual>
       <geometry>
@@ -65,5 +65,5 @@
   <joint name="base_imu_joint" type="fixed">
     <parent link="base_link" />
-    <child link="imu" />
+    <child link="imu_link" />
     <origin xyz="0.25 0 0.201" rpy="0 0 0" />
   </joint>

Commit message: Exclude collision detection for these components

File: ros_ws/src/navigation/config/karaburan.xacro (robot description, xacro)
@@ -28,6 +28,4 @@
       <material name="black" />
     </visual>
-    <collision>
-    </collision>
   </link>
   <link name="gps">
@@ -39,6 +37,4 @@
       <material name="black" />
     </visual>
-    <collision>
-    </collision>
   </link>
   <link name="lidar">

Commit message: Added innertia configuration

File: ros_ws/src/navigation/config/karaburan.xacro (robot description, xacro)
@@ -5,4 +5,15 @@
   </material>
   <link name="base_footprint" />
+  <!-- Box inertia (COM op link-origin) -->
+  <xacro:macro name="inertial_box" params="m x y z">
+    <inertial>
+      <origin xyz="0 0 0" rpy="0 0 0"/>
+      <mass value="${m}"/>
+      <inertia
+        ixx="${m*(y*y+z*z)/12.0}" ixy="0" ixz="0"
+        iyy="${m*(x*x+z*z)/12.0}" iyz="0"
+        izz="${m*(x*x+y*y)/12.0}"/>
+    </inertial>
+  </xacro:macro>
   <link name="base_link">
     <visual>
@@ -19,4 +30,5 @@
       <origin xyz="0 0 0.1" rpy="0 0 0" />
     </collision>
+    <xacro:inertial_box m="4.0" x="0.6" y="0.4" z="0.2" />
   </link>
   <link name="imu_link">

Commit message: Added launching of simulator. This simulator is funny: the bounce increases

File: ros_ws/src/navigation/config/karaburan.xacro (robot description, xacro)
@@ -1,12 +1,28 @@
 <?xml version="1.0" ?>
 <robot name="karaburan" xmlns:xacro="http://www.ros.org/wiki/xacro">
+  <xacro:property name="with_gazebo" default="false"/>
+  <xacro:property name="WITH_GAZEBO"
+    value="${str(with_gazebo).lower() in ['1','true','yes']}"/>
+  <xacro:if value="${WITH_GAZEBO}">
+    <gazebo>
+      <plugin name="hydrodynamics" filename="gz-sim-hydrodynamics-system">
+        <link_name>base_link</link_name>
+        <water_density>998</water_density>
+        <xU>80</xU><xUabsU>300</xUabsU>
+        <yV>80</yV><yVabsV>300</yVabsV>
+        <zW>300</zW><zWabsW>1500</zWabsW>
+        <kP>80</kP><kPabsP>300</kPabsP>
+        <mQ>80</mQ><mQabsQ>300</mQabsQ>
+        <nR>40</nR><nRabsR>200</nRabsR>
+      </plugin>
+    </gazebo>
+  </xacro:if>
   <material name="black">
      <color rgba="0.9 0.9 0.9 0.8" />
   </material>
-  <link name="base_footprint" />
   <!-- Box inertia (COM op link-origin) -->
   <xacro:macro name="inertial_box" params="m x y z">
     <inertial>
-      <origin xyz="0 0 0" rpy="0 0 0"/>
+      <origin xyz="0 0 ${z/2 + 0.01} " rpy="0 0 0"/>
       <mass value="${m}"/>
       <inertia
@@ -66,9 +82,4 @@
     </collision>
   </link>
-  <joint name="base_joint" type="fixed">
-    <parent link="base_footprint" />
-    <child link="base_link" />
-    <origin xyz="0 0 -0.1" rpy="0 0 0" />
-  </joint>
   <joint name="base_imu_joint" type="fixed">
     <parent link="base_link" />

Commit message: Trying to get a floating boat. Still failing

File: ros_ws/src/navigation/config/karaburan.xacro (robot description, xacro)
@@ -2,4 +2,5 @@
 <robot name="karaburan" xmlns:xacro="http://www.ros.org/wiki/xacro">
   <xacro:property name="with_gazebo" default="false"/>
+  <xacro:property name="hydro_link" value="base_foutprint"/>
   <xacro:property name="WITH_GAZEBO"
     value="${str(with_gazebo).lower() in ['1','true','yes']}"/>
@@ -7,12 +8,14 @@
     <gazebo>
       <plugin name="hydrodynamics" filename="gz-sim-hydrodynamics-system">
-        <link_name>base_link</link_name>
+        <link_name>${hydro_link}</link_name>
         <water_density>998</water_density>
-        <xU>80</xU><xUabsU>300</xUabsU>
-        <yV>80</yV><yVabsV>300</yVabsV>
-        <zW>300</zW><zWabsW>1500</zWabsW>
-        <kP>80</kP><kPabsP>300</kPabsP>
-        <mQ>80</mQ><mQabsQ>300</mQabsQ>
-        <nR>40</nR><nRabsR>200</nRabsR>
+        <disable_coriolis>true</disable_coriolis>
+        <disable_added_mass>true</disable_added_mass>
+        <xU>10</xU><xUabsU>60</xUabsU>
+        <yV>10</yV><yVabsV>60</yVabsV>-->
+        <zW>20</zW><!--zWabsW>1500</zWabsW-->
+        <kP>25</kP><kPabsP>80</kPabsP>
+        <mQ>50</mQ><mQabsQ>80</mQabsQ>
+        <nR>20</nR><nRabsR>60</nRabsR>-->
       </plugin>
     </gazebo>
@@ -24,5 +27,5 @@
   <xacro:macro name="inertial_box" params="m x y z">
     <inertial>
-      <origin xyz="0 0 ${z/2 + 0.01} " rpy="0 0 0"/>
+      <origin xyz="0 0 ${z*0.4}" rpy="0 0 0"/>
       <mass value="${m}"/>
       <inertia
@@ -32,4 +35,15 @@
     </inertial>
   </xacro:macro>
+  <xacro:macro name="inertial_cylinder_z" params="m r l">
+    <inertial>
+      <origin xyz="0 0 0" rpy="0 0 0"/>
+      <mass value="${m}"/>
+      <inertia
+        ixx="${m*(3*r*r + l*l)/12.0}" ixy="0" ixz="0"
+        iyy="${m*(3*r*r + l*l)/12.0}" iyz="0"
+        izz="${0.5*m*r*r}"/>
+    </inertial>
+  </xacro:macro>
+  <link name="base_footprint"/>
   <link name="base_link">
     <visual>
@@ -56,4 +70,10 @@
       <material name="black" />
     </visual>
+    <sensor name="imu_sensor" type="imu">
+      <always_on>1</always_on>
+      <update_rate>1</update_rate>
+      <visualize>true</visualize>
+      <topic>imu</topic>
+    </sensor>
   </link>
   <link name="gps">
@@ -81,5 +101,37 @@
       <material name="black" />
     </collision>
+    <sensor name="lidar" type="gpu_lidar">
+      <always_on>true</always_on>
+      <visualize>true</visualize>
+      <update_rate>5</update_rate>
+      <topic>scan</topic>
+      <gz_frame_id>lidar_link</gz_frame_id>
+      <lidar>
+        <scan>
+          <horizontal>
+            <samples>360</samples>
+            <resolution>1.000000</resolution>
+            <min_angle>0.000000</min_angle>
+            <max_angle>6.280000</max_angle>
+          </horizontal>
+        </scan>
+        <range>
+          <min>0.120000</min>
+          <max>3.5</max>
+          <resolution>0.015000</resolution>
+        </range>
+        <noise>
+          <type>gaussian</type>
+          <mean>0.0</mean>
+          <stddev>0.01</stddev>
+        </noise>
+      </lidar>
+    </sensor>
   </link>
+  <joint name="base_footprint_to_base_link" type="fixed">
+    <parent link="base_footprint"/>
+    <child link="base_link"/>
+    <origin xyz="0 0 0" rpy="0 0 0"/>
+  </joint>
   <joint name="base_imu_joint" type="fixed">
     <parent link="base_link" />
@@ -101,4 +153,5 @@
         <material name="black" />
       </visual>
+      <xacro:inertial_cylinder_z m="0.05" r="0.03" l="0.01"/>
     </link>
   </xacro:macro>

Commit message: Removing redundance xonfiguration

File: ros_ws/src/navigation/config/karaburan.xacro (robot description, xacro)
@@ -1,24 +1,4 @@
 <?xml version="1.0" ?>
 <robot name="karaburan" xmlns:xacro="http://www.ros.org/wiki/xacro">
-  <xacro:property name="with_gazebo" default="false"/>
-  <xacro:property name="hydro_link" value="base_foutprint"/>
-  <xacro:property name="WITH_GAZEBO"
-    value="${str(with_gazebo).lower() in ['1','true','yes']}"/>
-  <xacro:if value="${WITH_GAZEBO}">
-    <gazebo>
-      <plugin name="hydrodynamics" filename="gz-sim-hydrodynamics-system">
-        <link_name>${hydro_link}</link_name>
-        <water_density>998</water_density>
-        <disable_coriolis>true</disable_coriolis>
-        <disable_added_mass>true</disable_added_mass>
-        <xU>10</xU><xUabsU>60</xUabsU>
-        <yV>10</yV><yVabsV>60</yVabsV>-->
-        <zW>20</zW><!--zWabsW>1500</zWabsW-->
-        <kP>25</kP><kPabsP>80</kPabsP>
-        <mQ>50</mQ><mQabsQ>80</mQabsQ>
-        <nR>20</nR><nRabsR>60</nRabsR>-->
-      </plugin>
-    </gazebo>
-  </xacro:if>
   <material name="black">
      <color rgba="0.9 0.9 0.9 0.8" />

Commit message: More realistic dimensions for the boat

File: ros_ws/src/navigation/config/karaburan.xacro (robot description, xacro)
@@ -29,16 +29,16 @@
     <visual>
       <geometry>
-        <box size="0.6 0.4 0.2" />
+        <box size="0.5 0.25 0.13" />
       </geometry>
-      <origin xyz="0 0 0.1" rpy="0 0 0" />
+      <origin xyz="0 0 0.065" rpy="0 0 0" />
       <material name="black" />
     </visual>
     <collision>
       <geometry>
-        <box size="0.6 0.4 0.2" />
+        <box size="0.5 0.25 0.13" />
       </geometry>
-      <origin xyz="0 0 0.1" rpy="0 0 0" />
+      <origin xyz="0 0 0.065" rpy="0 0 0" />
     </collision>
-    <xacro:inertial_box m="4.0" x="0.6" y="0.4" z="0.2" />
+    <xacro:inertial_box m="2.0" x="0.5" y="0.25" z="0.13" />
   </link>
   <link name="imu_link">
@@ -117,10 +117,10 @@
     <parent link="base_link" />
     <child link="imu_link" />
-    <origin xyz="0.25 0 0.201" rpy="0 0 0" />
+    <origin xyz="0.23 0 0.131" rpy="0 0 0" />
   </joint>
   <joint name="base_gps_joint" type="fixed">
     <parent link="base_link" />
     <child link="gps" />
-    <origin xyz="-0.25 0 0.201" rpy="0 0 0" />
+    <origin xyz="-0.23 0 0.131" rpy="0 0 0" />
   </joint>
   <xacro:macro name="prop_link" params="prefix">
@@ -128,10 +128,10 @@
       <visual>
         <geometry>
-          <cylinder radius="0.04" length="0.025" />
+          <cylinder radius="0.025" length="0.01" />
         </geometry>
         <origin xyz="0 0 0" rpy="0 1.57 0" />
         <material name="black" />
       </visual>
-      <xacro:inertial_cylinder_z m="0.05" r="0.03" l="0.01"/>
+      <xacro:inertial_cylinder_z m="0.05" r="0.025" l="0.01"/>
     </link>
   </xacro:macro>
@@ -141,10 +141,10 @@
     <parent link="base_link" />
     <child link="lidar" />
-    <origin xyz="0 0 0.225" rpy="0 0 0" />
+    <origin xyz="0 0 0.155" rpy="0 0 0" />
   </joint>
   <joint name="base_left_prop_joint" type="continuous">
     <parent link="base_link" />
     <child link="left_prop" />
-    <origin xyz="-0.25 0.1 -0.045" rpy="0 0 0" />
+    <origin xyz="-0.25 0.09 -0.045" rpy="0 0 0" />
     <axis xyz="1 0 0" />
   </joint>
@@ -152,5 +152,5 @@
     <parent link="base_link" />
     <child link="right_prop" />
-    <origin xyz="-0.25 -0.1 -0.045" rpy="0 0 0" />
+    <origin xyz="-0.25 -0.09 -0.045" rpy="0 0 0" />
     <axis xyz="1 0 0" />
   </joint>

Commit message: Adding nav2 stack to the simulated launch

File: ros_ws/src/navigation/config/karaburan.xacro (robot description, xacro)
@@ -57,5 +57,5 @@
     </sensor>
   </link>
-  <link name="gps">
+  <link name="gps_link">
     <visual>
       <geometry>
@@ -121,5 +121,5 @@
   <joint name="base_gps_joint" type="fixed">
     <parent link="base_link" />
-    <child link="gps" />
+    <child link="gps_link" />
     <origin xyz="-0.23 0 0.131" rpy="0 0 0" />
   </joint>

Commit message: Starting something that accepts waypoints now works

File: ros_ws/src/navigation/config/karaburan.xacro (robot description, xacro)
@@ -25,5 +25,4 @@
     </inertial>
   </xacro:macro>
-  <link name="base_footprint"/>
   <link name="base_link">
     <visual>
@@ -109,9 +108,4 @@
     </sensor>
   </link>
-  <joint name="base_footprint_to_base_link" type="fixed">
-    <parent link="base_footprint"/>
-    <child link="base_link"/>
-    <origin xyz="0 0 0" rpy="0 0 0"/>
-  </joint>
   <joint name="base_imu_joint" type="fixed">
     <parent link="base_link" />

Commit message: Updating lidar link name

File: ros_ws/src/navigation/config/karaburan.xacro (robot description, xacro)
@@ -65,5 +65,5 @@
     </visual>
   </link>
-  <link name="lidar">
+  <link name="lidar_link">
     <visual>
       <geometry>
@@ -134,5 +134,5 @@
   <joint name="base_lidar_joint" type="fixed">
     <parent link="base_link" />
-    <child link="lidar" />
+    <child link="lidar_link" />
     <origin xyz="0 0 0.155" rpy="0 0 0" />
   </joint>
